Commit message: update import routine for CAD based import. add eef to robot urdf

File: iiwa_description/urdf/iiwa14_tool.urdf.xacro (robot description, xacro)
@@ -1,58 +1,35 @@
 <?xml version="1.0"?>
-<!-- Here we define the robot, we named it "iiwa7_tool" -->
-<robot xmlns:xacro="http://www.ros.org/wiki/xacro" name="iiwa7_tool">
+<!-- Here we define the robot, we named it "iiwa14_tool" -->
+<robot xmlns:xacro="http://www.ros.org/wiki/xacro" name="iiwa14_camera_light_eef">
   <!-- Import Rviz colors -->
   <xacro:include filename="$(find iiwa_description)/urdf/materials.xacro" />
-  <!--Import the iiwa7 macro -->
-  <xacro:include filename="$(find iiwa_description)/urdf/iiwa7.xacro"/>
-  <!--  Arguments for the iiwa7 macro  -->
+  <!--Import the iiwa14 macro -->
+  <xacro:include filename="$(find iiwa_description)/urdf/iiwa14.xacro"/>
+  <!--  Arguments for the iiwa14 macro  -->
   <xacro:arg name="hardware_interface" default="PositionJointInterface"/>
   <xacro:arg name="robot_name" default="iiwa"/>
-  <!--  Define the origin of your 3D space
-  Here we define a box lying at 0,0,0 with some dimensions, in reality our robot is place on top of a metal cart with those dimensions.
-  This will include the cart in the scene and avoid the robot to hit it when using MoveIt!
-  If you don't want to have that you can define a basic world link (see commented lines)
-  -->
-  <!--     <link name="world"/> -->
-  <link name="world">
-    <visual>
-      <origin xyz="0 0 0.42" rpy="0 0 0"/>
-      <geometry>
-	<box size="0.68 0.605 0.84"/>
-      </geometry>
-    </visual>
-    <collision>
-      <origin xyz="0 0 0.42" rpy="0 0 0"/>
-      <geometry>
-	<box size="0.68 0.605 0.84"/>
-      </geometry>
-    </collision>
-  </link>
-  <gazebo reference="world">
-    <static>true</static>
-  </gazebo>
-  <!-- Here we insert an iiwa7 robot in the scene, it's origin is just on top of the box previously defined. You can use 0,0,0 if you don't have that. -->
-  <xacro:iiwa7 hardware_interface="$(arg hardware_interface)" robot_name="$(arg robot_name)" parent="world">
-    <origin xyz="0 0 0.84" rpy="0 0 0"/>
-  </xacro:iiwa7>
+  <link name="world" />
+  <!-- Here we insert an iiwa14 robot in the scene, it's origin is just on top of the box previously defined. You can use 0,0,0 if you don't have that. -->
+  <xacro:iiwa14 hardware_interface="$(arg hardware_interface)" robot_name="$(arg robot_name)" parent="world">
+    <origin xyz="0 0 0" rpy="0 0 0" />
+  </xacro:iiwa14>
   <!-- Tool properties -->
-  <property name="tool_mass" value="0.200" />
-  <property name="tool_joint_offset" value="0.00 0.00 0.00" />
-  <property name="tool_link_offset" value="0.00 0.00 0.1275" />
-  <!--  Here we define a dummy joint between the tip of the iiwa7 and the base of the tool.
+  <xacro:property name="eef_mass" value="0.200" />
+  <xacro:property name="eef_joint_offset" value="0.00 0.00 0.00" />
+  <xacro:property name="eef_link_offset" value="0.00 0.00 0.12" />
+  <!--  Here we define a dummy joint between the tip of the iiwa14 and the base of the tool.
   There is no offset between the two, that means the tool is attached at the robot flange. -->
-  <joint name="tool_joint" type="fixed">
+  <joint name="eef_joint" type="fixed">
     <parent link="iiwa_link_ee" />
-    <child link = "tool_link" />
-    <origin xyz="${tool_joint_offset}" rpy="0 ${PI/2.0} 0" />
+    <child link = "eef_link" />
+    <origin xyz="${eef_joint_offset}" rpy="0 ${PI/2.0} 0" />
   </joint>
   <!-- Here we define the geometry of the tool. We designed the tool ourselves, so we have a mesh file that represents it.
   Else, one can define it using a geometric representation that approximate it, like a cylinder (see commented lines) -->
-  <link name="tool_link">
+  <link name="eef_link">
     <visual>
       <origin xyz="0 0 0" rpy="0 0 0"/>
       <geometry>
-	<mesh filename="package://iiwa_tool_description/meshes/visual/tool.stl"/>
-	<!-- 	<cylinder length="0.1275" radius="0.020"/> -->
+	      <mesh filename="/home/alexander/iiwa_stack_ws/src/iiwa_stack/iiwa_description/meshes/iiwa14/visual/prod_eef_assembly.stl"/>
       </geometry>
       <material name="Grey"/>
@@ -61,6 +38,5 @@
       <origin xyz="0 0 0" rpy="0 0 0"/>
       <geometry>
-	<mesh filename="package://iiwa_tool_description/meshes/visual/tool.stl"/>
-	<!-- 	<cylinder length="0.1275" radius="0.020"/> -->
+	      <mesh filename="/home/alexander/iiwa_stack_ws/src/iiwa_stack/iiwa_description/meshes/iiwa14/visual/prod_eef_assembly.stl"/>
       </geometry>
       <material name="Grey"/>
@@ -68,10 +44,10 @@
   </link>
   <!--  Here we define another dummy joint. It is placed at the end of the tool, so we can then attach a frame at its TCP for control -->
-  <joint name="tool_tip_joint" type="fixed">
-    <parent link="tool_link" />
-    <child link = "tool_link_ee" />
-    <origin xyz="${tool_link_offset}" rpy="0 0 0" />
+  <joint name="eef_tip_joint" type="fixed">
+    <parent link="eef_link" />
+    <child link = "eef_link_ee" />
+    <origin xyz="${eef_link_offset}" rpy="0 0 0" />
   </joint>
   <!--  The TCP frame is here defined -->
-  <link name="tool_link_ee"/>
+  <link name="eef_link_ee"/>
 </robot>
