Commit message: completed trajectory loop, adjusted robot position

File: iiwa_description/urdf/iiwa14.xacro (robot description, xacro)
@@ -72,5 +72,5 @@
           <mesh filename="package://iiwa_description/meshes/iiwa14/visual/link_1.stl"/>
         </geometry>
-        <material name="Orange"/>
+        <material name="Grey"/>
       </visual>
       <collision>
@@ -79,5 +79,5 @@
           <mesh filename="package://iiwa_description/meshes/iiwa14/collision/link_1.stl"/>
         </geometry>
-        <material name="Orange"/>
+        <material name="Grey"/>
       </collision>
     </link>
@@ -107,5 +107,5 @@
           <mesh filename="package://iiwa_description/meshes/iiwa14/visual/link_2.stl"/>
         </geometry>
-        <material name="Orange"/>
+        <material name="Grey"/>
       </visual>
       <collision>
@@ -114,5 +114,5 @@
           <mesh filename="package://iiwa_description/meshes/iiwa14/collision/link_2.stl"/>
         </geometry>
-        <material name="Orange"/>
+        <material name="Grey"/>
       </collision>
     </link>
@@ -142,5 +142,5 @@
           <mesh filename="package://iiwa_description/meshes/iiwa14/visual/link_3.stl"/>
         </geometry>
-        <material name="Orange"/>
+        <material name="Grey"/>
       </visual>
       <collision>
@@ -149,5 +149,5 @@
           <mesh filename="package://iiwa_description/meshes/iiwa14/collision/link_3.stl"/>
         </geometry>
-        <material name="Orange"/>
+        <material name="Grey"/>
       </collision>
     </link>
@@ -177,5 +177,5 @@
           <mesh filename="package://iiwa_description/meshes/iiwa14/visual/link_4.stl"/>
         </geometry>
-        <material name="Orange"/>
+        <material name="Grey"/>
       </visual>
       <collision>
@@ -184,5 +184,5 @@
           <mesh filename="package://iiwa_description/meshes/iiwa14/collision/link_4.stl"/>
         </geometry>
-        <material name="Orange"/>
+        <material name="Grey"/>
       </collision>
     </link>
@@ -212,5 +212,5 @@
           <mesh filename="package://iiwa_description/meshes/iiwa14/visual/link_5.stl"/>
         </geometry>
-        <material name="Orange"/>
+        <material name="Grey"/>
       </visual>
       <collision>
@@ -219,5 +219,5 @@
           <mesh filename="package://iiwa_description/meshes/iiwa14/collision/link_5.stl"/>
         </geometry>
-        <material name="Orange"/>
+        <material name="Grey"/>
       </collision>
     </link>
@@ -247,5 +247,5 @@
           <mesh filename="package://iiwa_description/meshes/iiwa14/visual/link_6.stl"/>
         </geometry>
-        <material name="Orange"/>
+        <material name="Grey"/>
       </visual>
       <collision>
@@ -254,5 +254,5 @@
           <mesh filename="package://iiwa_description/meshes/iiwa14/collision/link_6.stl"/>
         </geometry>
-        <material name="Orange"/>
+        <material name="Grey"/>
       </collision>
     </link>

File: iiwa_description/urdf/iiwa14_light_static.urdf.xacro (robot description, xacro)
@@ -12,4 +12,63 @@
   <xacro:arg name="origin_rpy" default="0 0 0" />
   <link name="world" />
+  <link name="table">
+    <visual>
+      <origin xyz="$(arg origin_xyz)" rpy="0 0 0" />
+      <geometry>
+        <box size="4 4 0.01"/>
+      </geometry>
+      <material name="Black" />
+    </visual>
+    <collision>
+      <origin xyz="$(arg origin_xyz)" rpy="0 0 0" />
+      <geometry>
+        <box size="4 4 0.01"/>
+      </geometry>
+    </collision>
+  </link>
+  <joint name="table_joint" type="fixed">
+    <parent link="world" />
+    <child link="table" />
+  </joint>
+  <link name="wall">
+    <visual>
+      <origin xyz="0 -1.35 0" rpy="0 0 0" />
+      <geometry>
+        <box size="4 0.01 4"/>
+      </geometry>
+      <material name="Black" />
+    </visual>
+    <collision>
+      <origin xyz="0 -1.35 0" rpy="0 0 0" />
+      <geometry>
+        <box size="4 0.01 4"/>
+      </geometry>
+    </collision>
+  </link>
+  <joint name="wall_joint" type="fixed">
+    <parent link="world" />
+    <child link="wall" />
+  </joint>
+  <!-- Error when loading the part stl file.
+  <link name="part">
+    <visual>
+      <origin xyz="0.25 3.45 0" rpy="0 0 ${-PI/2.0}" />
+      <geometry>
+        <mesh filename="/home/alexander/iiwa_stack_ws/src/iiwa_stack/iiwa_tesla/iiwa_tesla_publish/src/tesla_part_solo-1487454-03-B_neu (Meshed)002.stl"/>
+      </geometry>
+      <material name="Black" />
+    </visual>
+    <collision>
+      <origin xyz="0.25 3.45 0" rpy="0 0 ${-PI/2.0}" />
+      <geometry>
+        <mesh filename="/home/alexander/iiwa_stack_ws/src/iiwa_stack/iiwa_tesla/iiwa_tesla_publish/src/tesla_part_solo-1487454-03-B_neu (Meshed)002.stl"/>
+      </geometry>
+    </collision>
+  </link>
+  <joint name="part_joint" type="fixed">
+    <parent link="world" />
+    <child link="part" />
+  </joint>
+-->
   <!-- Here we insert an iiwa14 robot in the scene, it's origin is just on top of the box previously defined. You can use 0,0,0 if you don't have that. -->
   <xacro:iiwa14 hardware_interface="$(arg hardware_interface)" robot_name="$(arg robot_name)" parent="world">
