Commit message: start implementing box constraint

File: iiwa_description/urdf/iiwa14_light_static.urdf.xacro (robot description, xacro)
@@ -78,5 +78,5 @@
   <xacro:property name="eef_mass" value="0.200" />
   <xacro:property name="eef_joint_offset" value="0.00 0.00 0.00" />
-  <xacro:property name="eef_link_offset" value="0.00 0.00 0.12" />
+  <xacro:property name="eef_link_offset" value="0.00 0.00 0.190" />
   <!--  Here we define a dummy joint between the tip of the iiwa14 and the base of the tool.
   There is no offset between the two, that means the tool is attached at the robot flange. -->
@@ -90,5 +90,5 @@
   <link name="eef_link">
     <visual>
-      <origin xyz="0 0 0" rpy="0 0 0"/>
+      <origin xyz="0 0 0" rpy="0 0 ${PI/2}"/>
       <geometry>
 	      <mesh filename="package://iiwa_description/meshes/iiwa14/visual/prod_eef_assembly5_scaled_rebuild.stl"/>
@@ -97,5 +97,5 @@
     </visual>
     <collision>
-      <origin xyz="0 0 0" rpy="0 0 0"/>
+      <origin xyz="0 0 0" rpy="0 0 ${PI/2}"/>
       <geometry>
 	      <mesh filename="package://iiwa_description/meshes/iiwa14/visual/prod_eef_assembly5_scaled_rebuild.stl"/>

Commit message: try different kinematic solver. trac_ik preferred

File: iiwa_description/urdf/iiwa14_light_static.urdf.xacro (robot description, xacro)
@@ -33,5 +33,5 @@
   <link name="wall">
     <visual>
-      <origin xyz="0 -1.35 0" rpy="0 0 0" />
+      <origin xyz="0 -1.25 0" rpy="0 0 0" />
       <geometry>
         <box size="4 0.01 4"/>
@@ -40,5 +40,5 @@
     </visual>
     <collision>
-      <origin xyz="0 -1.35 0" rpy="0 0 0" />
+      <origin xyz="0 -1.25 0" rpy="0 0 0" />
       <geometry>
         <box size="4 0.01 4"/>
@@ -50,25 +50,4 @@
     <child link="wall" />
   </joint>
-  <!-- Error when loading the part stl file.
-  <link name="part">
-    <visual>
-      <origin xyz="0.25 3.45 0" rpy="0 0 ${-PI/2.0}" />
-      <geometry>
-        <mesh filename="/home/alexander/iiwa_stack_ws/src/iiwa_stack/iiwa_tesla/iiwa_tesla_publish/src/tesla_part_solo-1487454-03-B_neu (Meshed)002.stl"/>
-      </geometry>
-      <material name="Black" />
-    </visual>
-    <collision>
-      <origin xyz="0.25 3.45 0" rpy="0 0 ${-PI/2.0}" />
-      <geometry>
-        <mesh filename="/home/alexander/iiwa_stack_ws/src/iiwa_stack/iiwa_tesla/iiwa_tesla_publish/src/tesla_part_solo-1487454-03-B_neu (Meshed)002.stl"/>
-      </geometry>
-    </collision>
-  </link>
-  <joint name="part_joint" type="fixed">
-    <parent link="world" />
-    <child link="part" />
-  </joint>
--->
   <!-- Here we insert an iiwa14 robot in the scene, it's origin is just on top of the box previously defined. You can use 0,0,0 if you don't have that. -->
   <xacro:iiwa14 hardware_interface="$(arg hardware_interface)" robot_name="$(arg robot_name)" parent="world">

Commit message: add new eef, edit data metrics in notebook

File: iiwa_description/urdf/iiwa14_light_static.urdf.xacro (robot description, xacro)
@@ -55,7 +55,7 @@
   </xacro:iiwa14>
   <!-- Tool properties -->
-  <xacro:property name="eef_mass" value="0.200" />
+  <xacro:property name="eef_mass" value="6.000" />
   <xacro:property name="eef_joint_offset" value="0.00 0.00 0.00" />
-  <xacro:property name="eef_link_offset" value="0.00 0.00 0.190" />
+  <xacro:property name="eef_link_offset" value="0.00 0.00 0.250" />
   <!--  Here we define a dummy joint between the tip of the iiwa14 and the base of the tool.
   There is no offset between the two, that means the tool is attached at the robot flange. -->
@@ -71,5 +71,5 @@
       <origin xyz="0 0 0" rpy="0 0 ${PI/2}"/>
       <geometry>
-	      <mesh filename="package://iiwa_description/meshes/iiwa14/visual/prod_eef_assembly5_scaled_rebuild.stl"/>
+	      <mesh filename="package://iiwa_description/meshes/iiwa14/visual/primitive_model_230202-Body.stl"/>
       </geometry>
       <material name="Grey"/>
@@ -78,5 +78,5 @@
       <origin xyz="0 0 0" rpy="0 0 ${PI/2}"/>
       <geometry>
-	      <mesh filename="package://iiwa_description/meshes/iiwa14/visual/prod_eef_assembly5_scaled_rebuild.stl"/>
+	      <mesh filename="package://iiwa_description/meshes/iiwa14/visual/primitive_model_230202-Body.stl"/>
       </geometry>
       <material name="Grey"/>

Commit message: last rehearsal pt2

File: iiwa_description/urdf/iiwa14_light_static.urdf.xacro (robot description, xacro)
@@ -71,5 +71,5 @@
       <origin xyz="0 0 0" rpy="0 0 ${PI/2}"/>
       <geometry>
-	      <mesh filename="package://iiwa_description/meshes/iiwa14/visual/primitive_model_230202-Body.stl"/>
+	      <mesh filename="package://iiwa_description/meshes/iiwa14/visual/primitive_model_230202-Body_2.stl"/>
       </geometry>
       <material name="Grey"/>
@@ -78,5 +78,5 @@
       <origin xyz="0 0 0" rpy="0 0 ${PI/2}"/>
       <geometry>
-	      <mesh filename="package://iiwa_description/meshes/iiwa14/visual/primitive_model_230202-Body.stl"/>
+	      <mesh filename="package://iiwa_description/meshes/iiwa14/visual/primitive_model_230202-Body_2.stl"/>
       </geometry>
       <material name="Grey"/>
